Commit message: worked on robot

File: src/desktop_robot.urdf (robot description, URDF)
Before this commit: robot desktop_robot, 2 links, 1 joints
Links:
- added link fourth_link; visual box size=${fol_x} ${fol_y} ${fol_z}
- added link second_link; visual box size=${sel_x} ${sel_y} ${sel_z}
- added link third_link; visual box size=${thl_x} ${thl_y} ${thl_z}
- link base_link: geometry visual cylinder length=${base_z} radius=${base_r}
- link first_link: geometry visual box size=${fil_x} ${fil_y} ${fil_z}
Joints:
- removed joint base-fl_j
- added joint base-fil_j: type continuous, parent base_link, child first_link, origin xyz=0 0 ${base_z} rpy=0 0 0, axis 0 0 1
- added joint fil-sel_j: type continuous, parent first_link, child second_link, origin xyz=${fil_x/2} 0 ${fil_z} rpy=0 0 0, axis 0 1 0
- added joint sel-thl_j: type continuous, parent second_link, child third_link, origin xyz=${sel_x/2} 0 ${sel_z} rpy=0 0 0, axis 0 1 0
- added joint sl-thl_j: type continuous, parent third_link, child fourth_link, origin xyz=${thl_x/2} 0 ${thl_z} rpy=0 0 0, axis 0 0 1

Commit message: change readme

File: src/desktop_robot.urdf (robot description, URDF)
Before this commit: robot desktop_robot, 5 links, 4 joints
Links:
- added link fifth_link; visual box size=${ffl_x} ${ffl_y} ${ffl_z}

Commit message: worked on the robot!

File: src/desktop_robot.urdf (robot description, URDF)
Before this commit: robot desktop_robot, 6 links, 4 joints
Links:
- added link sixth_link; visual box size=${sil_x} ${sil_y} ${sil_z}
Joints:
- removed joint sl-thl_j
- added joint ffl-sil_j: type continuous, parent fifth_link, child sixth_link, origin xyz=0 0 ${sil_z/2} rpy=0 0 0, axis 0 0 1
- added joint fol-ffl_j: type continuous, parent fourth_link, child fifth_link, origin xyz=${fol_x/2} 0 ${fol_z} rpy=0 0 0, axis 0 0 1
- added joint thl-fol_j: type continuous, parent third_link, child fourth_link, origin xyz=${thl_x/2} 0 ${thl_z} rpy=0 0 0, axis 0 1 0
- joint sel-thl_j: origin xyz=${sel_x/2} 0 ${sel_z} rpy=0 0 0 -> xyz=0 ${sel_y} ${sel_z} rpy=0 0 0
