Commit message: lil changes to URDF, and started working with moveit!

File: src/desktop_robot.urdf.xacro (robot description, xacro)
@@ -4,22 +4,22 @@
 	<xacro:property name="base_r" value="0.5" />	<!-- base radius -->
 	<xacro:property name="base_z" value="0.1" />	<!-- base height -->
-	<xacro:property name="fil_y" value="0.7" />	<!-- first link width -->
-	<xacro:property name="fil_z" value="0.2" />	<!-- first link height -->
-	<xacro:property name="fil_x" value="0.7" />	<!-- first link depth -->
-	<xacro:property name="sel_y" value="0.2" />	<!-- second link width -->
-	<xacro:property name="sel_z" value="1" />	<!-- second link height -->
-	<xacro:property name="sel_x" value="0.1" />	<!-- second link depth -->
-	<xacro:property name="thl_y" value="0.2" />	<!-- third link width -->
-	<xacro:property name="thl_z" value="1" />	<!-- third link height -->
-	<xacro:property name="thl_x" value="0.1" />	<!-- third link depth -->
-	<xacro:property name="fol_y" value="0.2" />	<!-- fourth link width -->
-	<xacro:property name="fol_z" value="0.2" />	<!-- fourth link height -->
-	<xacro:property name="fol_x" value="0.2" />	<!-- fourth link depth -->
-	<xacro:property name="ffl_y" value="0.7" />	<!-- fifth link width -->
-	<xacro:property name="ffl_z" value="0.1" />	<!-- fifth link height -->
-	<xacro:property name="ffl_x" value="0.1" />	<!-- fifth link depth -->
-	<xacro:property name="sil_y" value="0.1" />	<!-- sixth link width -->
-	<xacro:property name="sil_z" value="1" />	<!-- sixth link height -->
-	<xacro:property name="sil_x" value="0.1" />	<!-- sixth link depth -->
+	<xacro:property name="fil_x" value="0.7" />	<!-- first link x -->
+	<xacro:property name="fil_y" value="0.7" />	<!-- first link y -->
+	<xacro:property name="fil_z" value="0.2" />	<!-- first link z -->
+	<xacro:property name="sel_x" value="0.1" />	<!-- second link x -->
+	<xacro:property name="sel_y" value="0.2" />	<!-- second link y -->
+	<xacro:property name="sel_z" value="1" />	<!-- second link z -->
+	<xacro:property name="thl_x" value="0.1" />	<!-- third link x -->
+	<xacro:property name="thl_y" value="0.2" />	<!-- third link y -->
+	<xacro:property name="thl_z" value="1" />	<!-- third link z -->
+	<xacro:property name="fol_x" value="0.1" />	<!-- fourth link x -->
+	<xacro:property name="fol_y" value="0.3" />	<!-- fourth link y -->
+	<xacro:property name="fol_z" value="0.1" />	<!-- fourth link z -->
+	<xacro:property name="ffl_x" value="0.1" />	<!-- fifth link x -->
+	<xacro:property name="ffl_y" value="0.2" />	<!-- fifth link y -->
+	<xacro:property name="ffl_z" value="0.05" />	<!-- fifth link z -->
+	<xacro:property name="sil_x" value="0.1" />	<!-- sixth link x -->
+	<xacro:property name="sil_y" value="0.1" />	<!-- sixth link y -->
+	<xacro:property name="sil_z" value="0.3" />	<!-- sixth link z -->
 	<!-- create here materials/colours -->
 	<material name="blue">
@@ -129,5 +129,5 @@
 	    <origin rpy="0 0 0" xyz="0 0 ${base_z}"/>
 	  </joint>
-	  <joint name="fil-sel_j" type="continuous">	<!-- create joint between base and first link-->
+	  <joint name="fil-sel_j" type="continuous">	<!-- create joint between first and second link-->
 	    <axis rpy="0 0 0" xyz="0 1 0"/>
 	    <parent link="first_link"/>
@@ -135,5 +135,5 @@
 	    <origin rpy="0 0 0" xyz="${fil_x/2} 0 ${fil_z}"/>
 	  </joint>
-	  <joint name="sel-thl_j" type="continuous">	<!-- create joint between base and first link-->
+	  <joint name="sel-thl_j" type="continuous">	<!-- create joint between second and third link-->
 	    <axis rpy="0 0 0" xyz="0 1 0"/>
 	    <parent link="second_link"/>
@@ -141,17 +141,17 @@
 	    <origin rpy="0 0 0" xyz="0 ${sel_y} ${sel_z}"/>
 	  </joint>
-	  <joint name="thl-fol_j" type="continuous">	<!-- create joint between base and first link-->
-	    <axis rpy="0 0 0" xyz="0 1 0"/>
+	  <joint name="thl-fol_j" type="continuous">	<!-- create joint between third and fourth link-->
+	    <axis rpy="0 0 0" xyz="0 0 1"/>
 	    <parent link="third_link"/>
 	    <child link="fourth_link"/>
 	    <origin rpy="0 0 0" xyz="${thl_x/2} 0 ${thl_z}"/>
 	  </joint>
-	  <joint name="fol-ffl_j" type="continuous">	<!-- create joint between base and first link-->
-		    <axis rpy="0 0 0" xyz="0 0 1"/>
+	  <joint name="fol-ffl_j" type="continuous">	<!-- create joint between fourth and fifth link-->
+		    <axis rpy="0 0 0" xyz="0 1 0"/>
 		    <parent link="fourth_link"/>
 		    <child link="fifth_link"/>
-		    <origin rpy="0 0 0" xyz="${fol_x/2} 0 ${fol_z}"/>
+		    <origin rpy="0 0 0" xyz="${fol_x/2} 0 ${fol_z/2}"/>
 	  </joint>
-	  <joint name="ffl-sil_j" type="continuous">	<!-- create joint between base and first link-->
+	  <joint name="ffl-sil_j" type="continuous">	<!-- create joint between fifth and sixth link-->
 		    <axis rpy="0 0 0" xyz="0 0 1"/>
 		    <parent link="fifth_link"/>
